File: boards/camp-front/camp-front.kicad_pcb (KiCad board)
At the start: 2 copper layers, 16 parts, among them J1 STEMMA, J2 VICTRON_0, J3 VICTRON_1, J4 PWR_MON, J5 WAGO 2601-1102, J7 WAGO 2601-3103, J8 WAGO 2601-3103, K1 EE2-5NU, K3 EE2-5NU, Q1 BC847W, Q4 BC847W, U1 RP2350-CAN

Commit message: Worked on boards
Parts:
- removed J4: PWR_MON, Connector_JST:JST_PH_B4B-PH-K_1x04_P2.00mm_Vertical
- added J6: TANK_SENSE, TerminalBlock_WAGO:TerminalBlock_WAGO_2601-1102_1x02_P3.50mm_Horizontal, F.Cu at (253.4, 106.4)
- added JP1: Jumper_3_Open, Connector_PinHeader_1.00mm:PinHeader_1x03_P1.00mm_Vertical, F.Cu at (157.8, 97.8)
- added Q3: IRF9Z24NPbF, Package_TO_SOT_THT:TO-220-3_Horizontal_TabDown, F.Cu at (237.2, 107.3)
- added Q5: BC847W, Package_TO_SOT_SMD:SOT-323_SC-70, F.Cu at (236.9, 111.1)
- added R39: 1k, Resistor_SMD:R_0805_2012Metric_Pad1.20x1.40mm_HandSolder, F.Cu at (231.8, 114.3)
- added R40: 1k, Resistor_SMD:R_0805_2012Metric_Pad1.20x1.40mm_HandSolder, F.Cu at (231.8, 112.4)
- added R41: 200, Resistor_SMD:R_0805_2012Metric_Pad1.20x1.40mm_HandSolder, F.Cu at (240.9, 106.7)
- added R42: 27k, Resistor_SMD:R_0805_2012Metric_Pad1.20x1.40mm_HandSolder, F.Cu at (240.9, 108.6)
- added R43: 10k, Resistor_SMD:R_0805_2012Metric_Pad1.20x1.40mm_HandSolder, F.Cu at (240.9, 110.5)
- added R44: 200, Resistor_SMD:R_0805_2012Metric_Pad1.20x1.40mm_HandSolder, F.Cu at (164.5, 101.0)
- added R45: 200, Resistor_SMD:R_0805_2012Metric_Pad1.20x1.40mm_HandSolder, F.Cu at (164.5, 113.7)
- added R46: 1k, Resistor_SMD:R_0805_2012Metric_Pad1.20x1.40mm_HandSolder, F.Cu at (144.1, 105.9)
- added R47: 1k, Resistor_SMD:R_0805_2012Metric_Pad1.20x1.40mm_HandSolder, F.Cu at (148.6, 106.0)
- added R48: 1k, Resistor_SMD:R_0805_2012Metric_Pad1.20x1.40mm_HandSolder, F.Cu at (148.6, 113.7)
- added R49: 1k, Resistor_SMD:R_0805_2012Metric_Pad1.20x1.40mm_HandSolder, F.Cu at (164.5, 108.6)
- added U2: TLP293-4, Package_SO:SOIC-16_4.55x10.3mm_P1.27mm, F.Cu at (157.5, 106.7)
- J2: value VICTRON_0 -> UART_0
- J3: value VICTRON_1 -> UART_1
- moved D7 69.5 mm to (213.4, 55.9)
- moved Q4 61.1 mm to (203.8, 56.5)
- moved D8 60.5 mm to (186.1, 55.9)
- moved Q1 58.2 mm to (192.4, 50.8)
- moved R37 53.4 mm to (207.6, 54.0)
- moved J3 43.9 mm to (169.1, 115.4), turned to 90 degrees
- moved R38 40.0 mm to (187.3, 52.1)
- moved J2 39.7 mm to (169.1, 104.0), turned to 90 degrees
Connections:
- J2 pad 1: unconnected-(J2-Pin_1-Pad1) -> /VE0_GND
- J2 pad 2: unconnected-(J2-Pin_2-Pad2) -> /VE0_TX_H
- J2 pad 3: unconnected-(J2-Pin_3-Pad3) -> /VE0_RX_H
- J2 pad 4: unconnected-(J2-Pin_4-Pad4) -> /VE0_V+
- J3 pad 1: unconnected-(J3-Pin_1-Pad1) -> /SER1_GND
- J3 pad 2: unconnected-(J3-Pin_2-Pad2) -> /SER1_TX_H
- J3 pad 3: unconnected-(J3-Pin_3-Pad3) -> /SER1_RX_H
- J3 pad 4: unconnected-(J3-Pin_4-Pad4) -> /SER1_V+
