File: boards/camp-front/camp-front.kicad_sch (KiCad schematic)
At the start: 16 parts, among them J1 STEMMA, J2 VICTRON_0, J3 VICTRON_1, J4 PWR_MON, J5 WAGO 2601-1102, J7 WAGO 2601-3103, J8 WAGO 2601-3103, K1 EE2-5NU, K3 EE2-5NU, Q1 BC847W, Q4 BC847W, U1 RP2350-CAN

Commit message: Worked on boards
Parts:
- removed J4: PWR_MON, Connector_JST:JST_PH_B4B-PH-K_1x04_P2.00mm_Vertical, symbol Connector_Generic:Conn_01x04
- added J6: TANK_SENSE, TerminalBlock_WAGO:TerminalBlock_WAGO_2601-1102_1x02_P3.50mm_Horizontal, symbol Connector:Screw_Terminal_01x02
- added JP1: Jumper_3_Open, Connector_PinHeader_1.00mm:PinHeader_1x03_P1.00mm_Vertical, symbol Jumper:Jumper_3_Open
- added Q3: IRF9Z24NPbF, Package_TO_SOT_THT:TO-220-3_Horizontal_TabDown, symbol Transistor_FET:Q_PMOS_GDSD
- added Q5: BC847W, Package_TO_SOT_SMD:SOT-323_SC-70, symbol Transistor_BJT:BC847W
- added R39, R40, R46, R47, R48, R49: 1k, Resistor_SMD:R_0805_2012Metric_Pad1.20x1.40mm_HandSolder, symbol Device:R_Small
- added R41, R44, R45: 200, Resistor_SMD:R_0805_2012Metric_Pad1.20x1.40mm_HandSolder, symbol Device:R_Small
- added R42: 27k, Resistor_SMD:R_0805_2012Metric_Pad1.20x1.40mm_HandSolder, symbol Device:R_Small
- added R43: 10k, Resistor_SMD:R_0805_2012Metric_Pad1.20x1.40mm_HandSolder, symbol Device:R_Small
- added U2: TLP293-4, Package_SO:SOIC-16_4.55x10.3mm_P1.27mm, symbol Isolator:TLP293-4
- J2: value VICTRON_0 -> UART_0
- J3: value VICTRON_1 -> UART_1
Connections:
- net +5V: now also JP1.3 (B)
- net GND: now also J6.2 (Pin_2), Q5.2 (E), R43.1, R47.1, R48.1, U2.2, U2.6
- net VE0_GND: now reaches J2.1 (Pin_1)
- net VE0_GND: now also R46.2, U2.4
- net VE0_TX_H: now reaches J2.2 (Pin_2)
- net VE0_TX_H: now also R46.1, U2.15
- net VE0_RX_H: now reaches J2.3 (Pin_3)
- net VE0_RX_H: now also R44.2
- net VE0_V+: now reaches J2.4 (Pin_4)
- net VE0_V+: now also JP1.2 (C), U2.16
- net SER1_GND: now reaches J3.1 (Pin_1)
- net SER1_GND: now also R49.2, U2.8
- net SER1_TX_H: now reaches J3.2 (Pin_2)
- net SER1_TX_H: now also R49.1, U2.11
- net SER1_RX_H: now reaches J3.3 (Pin_3)
- net SER1_RX_H: now also R45.2
- net SER1_V+: now reaches J3.4 (Pin_4)
- net SER1_V+: now also U2.12
- new net: R44.1, U2.3
- new net: J6.1 (Pin_1), R41.2, R42.2
- new net: Q3.3 (S), R41.1
- new net: Q3.1 (G), Q5.3 (C), R40.1
- new net: Q5.1 (B), R39.2
- new net: R45.1, U2.7
- new net +12V: Q3.2 (D), Q3.4 (D), R40.2
- new net +3V3: JP1.1 (A), U2.10, U2.14
- new net RX0: R47.2, U2.13
- new net RX1: R48.2, U2.9
- new net TANK_READ: R42.1, R43.2
- new net TANK_WRITE: R39.1
- new net TX0: U2.1
- new net TX1: U2.5
Other:
- moved on the sheet: D7, D8, J1, J2, J3, J5, J7, J8, K1, K3, Q1, Q4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
